Commit message: quad desc

File: ignition_ros2_control_demo/robot_demo_description/urdf/quadbot_description.urdf.xacro (robot description, xacro)
@@ -1,9 +1,9 @@
 <?xml version="1.0"?>
 <robot xmlns:xacro="http://www.ros.org/wiki/xacro">
-  <xacro:macro name="diffbot" params="prefix">
+  <xacro:macro name="quadbot" params="prefix">
   <!-- Constants for robot dimensions -->
   <xacro:property name="PI" value="3.1415926535897931"/>
   <xacro:property name="base_mass" value="0.6" /> <!-- arbitrary value for base mass -->
-  <xacro:property name="base_width" value="0.2" />
+  <xacro:property name="base_width" value="0.4" />
   <xacro:property name="base_length" value="0.2" />
   <xacro:property name="base_height" value="0.1" />
@@ -38,21 +38,36 @@
       </inertial>
     </link>
-    <joint name="${prefix}front_wheel_joint" type="continuous">
-      <parent link="${prefix}base_link"/>
-      <child link="${prefix}left_wheel"/>
-      <origin xyz="0 -${base_width/2} ${z_offset}" rpy="0 0 0"/>
-      <axis xyz="0 1 0"/>
-      <dynamics damping="0.2"/>
-    </joint>
-    <!-- left wheel Link -->
-    <link name="${prefix}left_wheel">
-      <collision>
-        <origin xyz="0 0 0" rpy="${PI/2} 0 0"/>
-        <geometry>
-          <cylinder length="${wheel_len}" radius="${wheel_radius}"/>
-        </geometry>
-      </collision>
-      <visual>
-        <origin xyz="0 0 0" rpy="${PI/2} 0 0"/>
+    <joint name="${prefix}front_wheel_hinge_joint" type="revolute">
+      <parent link="${prefix}base_link"/>
+      <child link="${prefix}front_wheel_hinge"/>
+      <origin xyz="${base_width/3} 0 ${z_offset}" rpy="0 ${PI/2} 0"/>
+      <axis xyz="-1 0 0"/>
+      <dynamics damping="0.2"/>
+      <limit lower="-${PI/2}" upper="${PI/2}" effort="1000" velocity="100" />
+    </joint>
+    <link name="${prefix}front_wheel_hinge">
+      <visual>
+        <origin xyz="0 0 0" rpy="0 0 0"/>
+        <geometry>
+          <sphere radius="${caster_wheel_radius/2}"/>
+        </geometry>
+        <material name="white"/>
+      </visual>
+      <inertial>
+        <origin xyz="0 0 0" rpy="0 0 0"/>
+        <mass value="0.100"/>
+        <inertia ixx="4E-06" ixy="0" ixz="0" iyy="4E-06" iyz="0" izz="4E-06"/>
+      </inertial>
+    </link>
+    <!-- front wheel Link -->
+    <link name="${prefix}front_wheel">
+      <collision>
+        <origin xyz="0 0 0" rpy="0 0 0"/>
+        <geometry>
+          <cylinder length="${wheel_len}" radius="${wheel_radius}"/>
+        </geometry>
+      </collision>
+      <visual>
+        <origin xyz="0 0 0" rpy="0 0 0"/>
         <geometry>
           <cylinder length="${wheel_len}" radius="${wheel_radius}"/>
@@ -61,5 +76,5 @@
       </visual>
       <inertial>
-        <origin xyz="0 0 0" rpy="${PI/2} 0 0"/>
+        <origin xyz="0 0 0" rpy="0 0 0"/>
         <mass value="${wheel_mass}"/>
         <inertia
@@ -67,23 +82,45 @@
           iyy="${wheel_mass / 12.0 * wheel_radius*wheel_radius}" iyz="0.0"
           izz="${wheel_mass / 12.0 * wheel_radius*wheel_radius}"/>
-        </inertial>
-      </link>
-    <joint name="${prefix}right_wheel_joint" type="continuous">
-      <parent link="${prefix}base_link"/>
-      <child link="${prefix}right_wheel"/>
-      <origin xyz="0 ${base_width/2} ${z_offset}" rpy="0 0 0"/>
-      <axis xyz="0 1 0"/>
-      <dynamics damping="0.2"/>
-    </joint>
-    <!-- right wheel Link -->
-    <link name="${prefix}right_wheel">
-      <collision>
-        <origin xyz="0 0 0" rpy="${PI/2} 0 0"/>
-        <geometry>
-          <cylinder length="${wheel_len}" radius="${wheel_radius}"/>
-        </geometry>
-      </collision>
-      <visual>
-        <origin xyz="0 0 0" rpy="${PI/2} 0 0"/>
+      </inertial>
+    </link>
+    <joint name="${prefix}front_wheel_joint" type="continuous">
+      <parent link="${prefix}front_wheel_hinge"/>
+      <child link="${prefix}front_wheel"/>
+      <origin xyz="0 0 0" rpy="${PI/2} 0 0"/>
+      <axis xyz="0 0 -1"/>
+      <dynamics damping="0.2"/>
+    </joint>
+    <joint name="${prefix}rear_wheel_hinge_joint" type="revolute">
+      <parent link="${prefix}base_link"/>
+      <child link="${prefix}rear_wheel_hinge"/>
+      <origin xyz="-${base_width/3} 0 ${z_offset}" rpy="0 ${PI/2} 0"/>
+      <axis xyz="-1 0 0"/>
+      <dynamics damping="0.2"/>
+      <limit lower="-${PI/2}" upper="${PI/2}" effort="1000" velocity="100" />
+    </joint>
+    <link name="${prefix}rear_wheel_hinge">
+      <visual>
+        <origin xyz="0 0 0" rpy="0 0 0"/>
+        <geometry>
+          <sphere radius="${caster_wheel_radius/2}"/>
+        </geometry>
+        <material name="white"/>
+      </visual>
+      <inertial>
+        <origin xyz="0 0 0" rpy="0 0 0"/>
+        <mass value="0.100"/>
+        <inertia ixx="4E-06" ixy="0" ixz="0" iyy="4E-06" iyz="0" izz="4E-06"/>
+      </inertial>
+    </link>
+    <!-- rear wheel Link -->
+    <link name="${prefix}rear_wheel">
+      <collision>
+        <origin xyz="0 0 0" rpy="0 0 0"/>
+        <geometry>
+          <cylinder length="${wheel_len}" radius="${wheel_radius}"/>
+        </geometry>
+      </collision>
+      <visual>
+        <origin xyz="0 0 0" rpy="0 0 0"/>
         <geometry>
           <cylinder length="${wheel_len}" radius="${wheel_radius}"/>
@@ -92,5 +129,5 @@
       </visual>
       <inertial>
-        <origin xyz="0 0 0" rpy="${PI/2} 0 0"/>
+        <origin xyz="0 0 0" rpy="0 0 0"/>
         <mass value="${wheel_mass}"/>
         <inertia
@@ -98,13 +135,14 @@
           iyy="${wheel_mass / 12.0 * wheel_radius*wheel_radius}" iyz="0.0"
           izz="${wheel_mass / 12.0 * wheel_radius*wheel_radius}"/>
-        </inertial>
-      </link>
-    <joint name="${prefix}caster_frontal_wheel_joint" type="fixed">
-      <parent link="${prefix}base_link"/>
-      <child link="${prefix}caster_frontal_wheel"/>
-      <origin xyz="${base_width/2 - caster_wheel_radius} 0 ${z_offset}" rpy="0 0 0"/>
-    </joint>
-    <!-- caster frontal wheel Link -->
-    <link name="${prefix}caster_frontal_wheel">
+      </inertial>
+    </link>
+    <joint name="${prefix}rear_wheel_joint" type="continuous">
+      <parent link="${prefix}rear_wheel_hinge"/>
+      <child link="${prefix}rear_wheel"/>
+      <origin xyz="0 0 0" rpy="${PI/2} 0 0"/>
+      <axis xyz="0 0 -1"/>
+      <dynamics damping="0.2"/>
+    </joint>
+    <link name="${prefix}caster_left_wheel">
       <collision>
         <origin xyz="0 0 0" rpy="0 0 0"/>
@@ -127,13 +165,12 @@
           iyy="${caster_wheel_mass * 0.4 * (caster_wheel_radius * caster_wheel_radius)}" iyz="0.0"
           izz="${caster_wheel_mass * 0.4 * (caster_wheel_radius * caster_wheel_radius)}"/>
-        </inertial>
-      </link>
-    <joint name="${prefix}caster_rear_wheel_joint" type="fixed">
-      <parent link="${prefix}base_link"/>
-      <child link="${prefix}caster_rear_wheel"/>
-      <origin xyz="${-base_width/2 + caster_wheel_radius} 0 ${z_offset}" rpy="0 0 0"/>
-    </joint>
-    <!-- caster rear wheel Link -->
-    <link name="${prefix}caster_rear_wheel">
+      </inertial>
+    </link>
+    <joint name="${prefix}caster_left_wheel_joint" type="fixed">
+      <parent link="${prefix}base_link"/>
+      <child link="${prefix}caster_left_wheel"/>
+      <origin xyz="0 ${base_length/2 - caster_wheel_radius} ${z_offset}" rpy="0 0 0"/>
+    </joint>
+    <link name="${prefix}caster_right_wheel">
       <collision>
         <origin xyz="0 0 0" rpy="0 0 0"/>
@@ -156,6 +193,11 @@
           iyy="${caster_wheel_mass * 0.4 * (caster_wheel_radius * caster_wheel_radius)}" iyz="0.0"
           izz="${caster_wheel_mass * 0.4 * (caster_wheel_radius * caster_wheel_radius)}"/>
-        </inertial>
-      </link>
+      </inertial>
+    </link>
+    <joint name="${prefix}caster_right_wheel_joint" type="fixed">
+      <parent link="${prefix}base_link"/>
+      <child link="${prefix}caster_right_wheel"/>
+      <origin xyz="0 -${base_length/2 - caster_wheel_radius} ${z_offset}" rpy="0 0 0"/>
+    </joint>
   </xacro:macro>
 </robot>
